Commit message: added/verified stuff

File: lidar_transforms/urdf/lidar_bench.urdf (robot description, URDF)
Before this commit: robot lidar_bench, 5 links, 4 joints
Links:
- removed link cart_base
- removed link laser_link
- added link hesai_lidar
Joints:
- removed joint laser_link_joint
- removed joint map_to_cart
- removed joint motor_joint
- added joint hesai_lidar_joint: type fixed, parent motor_axis, child hesai_lidar, origin xyz=0.0 0.0 0.09 rpy=0.0 0.0 -1.5708
- added joint map_to_motor: type continuous, parent map, child motor_axis, origin xyz=0.0 0.0 0.9406 rpy=0.0 0.0 0.0, axis 0 0 1

Commit message: Aarush/lidar reporting refactor (#2)
sTUFF

---------

Co-authored-by: Aarush Jain <aarush@polymathrobotics.com>

File: lidar_transforms/urdf/lidar_bench.urdf (robot description, URDF)
Before this commit: robot lidar_bench, 5 links, 4 joints
Links:
- removed link black_half_cylinder
- removed link cart_base
- added link white_wall; visual box size=0.0 2.4638 1.0287
Joints:
- removed joint map_to_black_half_cylinder
- removed joint map_to_cart
- removed joint motor_joint
- added joint map_to_motor: type continuous, parent map, child motor_axis, origin xyz=0.0 0.0 0.9406 rpy=0.0 0.0 0.0, axis 0 0 1
- added joint map_to_white_wall: type fixed, parent map, child white_wall, origin xyz=4.9276 0.0 1.07315 rpy=0.0 0.0 0.0
- joint hesai_lidar_joint: origin xyz=0.0 0.0 0.09 rpy=0.0 -1.5708 -1.5708 -> xyz=0.0 0.0 0.09 rpy=0.0 0.0 -1.5708

Commit message: added stuff

File: lidar_transforms/urdf/lidar_bench.urdf (robot description, URDF)
Before this commit: robot lidar_bench, 4 links, 3 joints
Links:
- link white_wall: geometry visual box size=0.0 1.2446 1.3716
Joints:
- joint map_to_white_wall: origin xyz=4.9276 0.0 1.07315 rpy=0.0 0.0 0.0 -> xyz=4.064 0.0 0.93218 rpy=0.0 0.0 0.0

Commit message: fixed polyview

File: lidar_transforms/urdf/lidar_bench.urdf (robot description, URDF)
Before this commit: robot lidar_bench, 4 links, 3 joints
Links:
- removed link white_wall
- added link blue_wall; visual box size=0.0 1.27 1.27
Joints:
- removed joint map_to_white_wall
- added joint map_to_blue_wall: type fixed, parent map, child blue_wall, origin xyz=3.048 0.0 0.889 rpy=0.0 0.0 0.0

Commit message: added folder for environment configs and lidar drivers

File: lidar_transforms/urdf/lidar_bench.urdf (robot description, URDF)
Before this commit: robot lidar_bench, 4 links, 3 joints
Links:
- removed link blue_wall
- removed link hesai_lidar
- added link white_wall; visual box size=0.0 1.2446 1.3716
- added link zadar
Joints:
- removed joint hesai_lidar_joint
- removed joint map_to_blue_wall
- added joint map_to_white_wall: type fixed, parent map, child white_wall, origin xyz=4.064 0.0 0.93218 rpy=0.0 0.0 0.0
- added joint zadar_joint: type fixed, parent motor_axis, child zadar, origin xyz=0.0 0.0 0.1016 rpy=0.0 0.0 0.0
